File: import/vacuum-stand.kicad_sch (KiCad schematic)
At the start: 75 parts, among them U1 МР248, U2 Диммер 2 канала, U3 ZMPT101B, U4 TCA9548A, X10 МР248 турбины 1, X11 МР248 турбины 2, X12 Диммер 2 канала, X13 ZMPT101B, X14 TCA9548A, X15 BME280, X16 DS18B20 №1, X17 DS18B20 №2, X18 Холл 1, X19 Холл 2, X20 Экран ILI9488, X21 Карта экрана, X9 Запас

Commit message: Стенд: штуцеры MPX5100DP — камера на P2, P1 в воздух
По даташиту NXP (раздел 4.1) P1 — сторона с надписью и давление на P1
должно быть больше: при трубке от бака на P1 датчик показывал бы ноль.
Описание датчика в stand.ts исправлено, файлы import/vacuum-stand*
пересозданы (STAND_WRITE=1).

Co-Authored-By: Claude Opus 5.5 <noreply@anthropic.com>
Claude-Session: https://claude.ai/code/session_01GQJVfWNfPicx79rJ5RavRD
Parts:
- B1: Описание Разрежение в баке 0–100 кПа: P1 — трубка к баку, P2 — откры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 -> Разрежение в баке 0–100 кПа: датчик меряет P1 − P2 (P1 > P2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
Changed lines of the file:
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@@
     (property "Datasheet" "" (id 3) (at 379.73 40.64 0) (effects (font (size 1.27 1.27)) hide))
     (property "Раздел" "Давление" (id 4) (at 379.73 40.64 0) (effects (font (size 1.27 1.27)) hide))
-    (property "Описание" "Разрежение в баке 0–100 кПа: P1 — трубка к баку, P2 — открыт в атмосферу (через ватку от пыли). Выход 0,2–4,7 В" (id 5) (at 379.73 40.64 0) (effects (font (size 1.27 1.27)) hide))
+    (property "Описание" "Разрежение в баке 0–100 кПа: датчик меряет P1 − P2 (P1 > P2), поэтому P2 (штуцер на стороне без надписи) — трубка к баку, P1 (сторона с надписью) — открыт в атмосферу (через ватку от пыли). Выход 0,2–4,7 В" (id 5) (at 379.73 40.64 0) (effects (font (size 1.27 1.27)) hide))
     (pin "1")
     (pin "2")
